Commit message: simplify loading the rg6

File: onrobot_rg_description/urdf/onrobot_rg6_model_macro.xacro (robot description, xacro)
@@ -3,4 +3,34 @@
   <xacro:include filename="$(find onrobot_rg_description)/urdf/onrobot_rg6_transmission.xacro" />
   <xacro:include filename="$(find onrobot_rg_description)/urdf/onrobot_rg6_gazebo.xacro" />
+  <xacro:macro name="onrobot_rg6_base_link" params="prefix">
+    <link name="${prefix}onrobot_rg6_base_link">
+      <inertial>
+        <origin xyz="0.0 0.0 0.0" rpy="0 0 0" />
+        <mass value="0.7" />
+        <inertia ixx="1.0E-03" ixy="1.0E-06" ixz="1.0E-06" iyy="1.0E-03" iyz="1.0E-06" izz="1.0E-03" />
+      </inertial>
+      <visual>
+        <origin xyz="0 0 0" rpy="0 0 0" />
+        <geometry>
+          <mesh filename="package://onrobot_rg_description/meshes/rg6/visual/base_link.stl" />
+        </geometry>
+        <material name="">
+          <color rgba="0.8 0.8 0.8 1" />
+        </material>
+      </visual>
+      <collision>
+        <origin xyz="0 0 0" rpy="0 0 0" />
+        <geometry>
+          <mesh filename="package://onrobot_rg_description/meshes/rg6/collision/base_link.stl" />
+        </geometry>
+      </collision>
+    </link>
+    <gazebo reference="${prefix}onrobot_rg6_base_link">
+      <mu1>1.0</mu1>
+      <mu2>1.0</mu2>
+      <selfCollide>false</selfCollide>
+      <material>Gazebo/White</material>
+    </gazebo>
+  </xacro:macro>
   <xacro:macro name="outer_knuckle" params="prefix fingerprefix">
     <link name="${prefix}${fingerprefix}_outer_knuckle">
@@ -116,5 +146,4 @@
     </joint>
   </xacro:macro>
-  <xacro:include filename="$(find onrobot_rg_description)/urdf/onrobot_rg6.xacro" />
   <xacro:macro name="finger_joint" params="prefix">
     <joint name="${prefix}finger_joint" type="revolute">
@@ -138,4 +167,13 @@
     <xacro:finger_joints prefix="${prefix}" fingerprefix="right" reflect="-1.0"/>
   </xacro:macro>
+  <xacro:macro name="finger_joints" params="prefix fingerprefix reflect">
+    <xacro:inner_knuckle_joint prefix="${prefix}" fingerprefix="${fingerprefix}" reflect="${reflect}"/>
+    <xacro:inner_finger_joint prefix="${prefix}" fingerprefix="${fingerprefix}"/>
+  </xacro:macro>
+  <xacro:macro name="finger_links" params="prefix fingerprefix">
+    <xacro:outer_knuckle prefix="${prefix}" fingerprefix="${fingerprefix}"/>
+    <xacro:inner_knuckle prefix="${prefix}" fingerprefix="${fingerprefix}"/>
+    <xacro:inner_finger prefix="${prefix}" fingerprefix="${fingerprefix}"/>
+  </xacro:macro>
   <xacro:macro name="onrobot_rg6" params="prefix">
     <xacro:onrobot_rg6_base_link prefix="${prefix}"/>

Commit message: add a grip target frame for motion planning

File: onrobot_rg_description/urdf/onrobot_rg6_model_macro.xacro (robot description, xacro)
@@ -176,4 +176,12 @@
     <xacro:inner_finger prefix="${prefix}" fingerprefix="${fingerprefix}"/>
   </xacro:macro>
+  <xacro:macro name="grip_target_frame" params="prefix">
+    <joint name="${prefix}grip_target_frame_joint" type="fixed">
+      <origin xyz="0 0 0.25" rpy="0 0 0" />
+      <parent link="${prefix}onrobot_rg6_base_link" />
+      <child link="${prefix}grip_target_frame" />
+    </joint>
+    <link name="${prefix}grip_target_frame"/>
+  </xacro:macro>
   <xacro:macro name="onrobot_rg6" params="prefix">
     <xacro:onrobot_rg6_base_link prefix="${prefix}"/>
@@ -184,4 +192,5 @@
     <xacro:onrobot_rg6_transmission prefix="${prefix}"/>
     <xacro:onrobot_rg6_gazebo prefix="${prefix}"/>
+    <xacro:grip_target_frame prefix="${prefix}"/>
   </xacro:macro>
 </robot>
