Commit message: First commit MM

File: onrobot_rg_description/urdf/onrobot_rg6.xacro (robot description, xacro)
@@ -1,6 +1,6 @@
 <?xml version="1.0"?>
 <robot xmlns:xacro="http://ros.org/wiki/xacro">
-  <xacro:macro name="onrobot_rg2_base_link" params="prefix">
-    <link name="${prefix}onrobot_rg2_base_link">
+  <xacro:macro name="onrobot_rg6_base_link" params="prefix">
+    <link name="${prefix}onrobot_rg6_base_link">
       <inertial>
         <origin xyz="0.0 0.0 0.0" rpy="0 0 0" />
@@ -11,5 +11,5 @@
         <origin xyz="0 0 0" rpy="0 0 0" />
         <geometry>
-          <mesh filename="package://onrobot_rg_description/meshes/rg2/visual/base_link.stl" />
+          <mesh filename="package://onrobot_rg_description/meshes/rg6/visual/base_link.stl" />
         </geometry>
         <material name="">
@@ -20,20 +20,20 @@
         <origin xyz="0 0 0" rpy="0 0 0" />
         <geometry>
-          <mesh filename="package://onrobot_rg_description/meshes/rg2/collision/base_link.stl" />
+          <mesh filename="package://onrobot_rg_description/meshes/rg6/collision/base_link.stl" />
         </geometry>
       </collision>
     </link>
-    <!-- <link name="flange"/>
-    <joint name="rg2_TM_joint" type="fixed">
-        <parent link="flange"/>
-        <child link="${prefix}onrobot_rg2_base_link"/>
+    <link name="world"/>
+    <joint name="joint0" type="fixed">
+        <parent link="world"/>
+        <child link="${prefix}onrobot_rg6_base_link"/>
         <origin xyz= "0. 0. 0." rpy="0. 0. 0." />
     </joint>
-    <gazebo reference="${prefix}onrobot_rg2_base_link">
+    <gazebo reference="${prefix}onrobot_rg6_base_link">
       <mu1>1.0</mu1>
       <mu2>1.0</mu2>
       <selfCollide>false</selfCollide>
       <material>Gazebo/White</material>
-    </gazebo> -->
+    </gazebo>
   </xacro:macro>
   <xacro:macro name="finger_joints" params="prefix fingerprefix reflect">

File: onrobot_rg_description/urdf/onrobot_rg6_model_macro.xacro (robot description, xacro)
@@ -3,34 +3,4 @@
   <xacro:include filename="$(find onrobot_rg_description)/urdf/onrobot_rg6_transmission.xacro" />
   <xacro:include filename="$(find onrobot_rg_description)/urdf/onrobot_rg6_gazebo.xacro" />
-  <xacro:macro name="onrobot_rg6_base_link" params="prefix">
-    <link name="${prefix}onrobot_rg6_base_link">
-      <inertial>
-        <origin xyz="0.0 0.0 0.0" rpy="0 0 0" />
-        <mass value="0.7" />
-        <inertia ixx="1.0E-03" ixy="1.0E-06" ixz="1.0E-06" iyy="1.0E-03" iyz="1.0E-06" izz="1.0E-03" />
-      </inertial>
-      <visual>
-        <origin xyz="0 0 0" rpy="0 0 0" />
-        <geometry>
-          <mesh filename="package://onrobot_rg_description/meshes/rg6/visual/base_link.stl" />
-        </geometry>
-        <material name="">
-          <color rgba="0.8 0.8 0.8 1" />
-        </material>
-      </visual>
-      <collision>
-        <origin xyz="0 0 0" rpy="0 0 0" />
-        <geometry>
-          <mesh filename="package://onrobot_rg_description/meshes/rg6/collision/base_link.stl" />
-        </geometry>
-      </collision>
-    </link>
-    <gazebo reference="${prefix}onrobot_rg6_base_link">
-      <mu1>1.0</mu1>
-      <mu2>1.0</mu2>
-      <selfCollide>false</selfCollide>
-      <material>Gazebo/White</material>
-    </gazebo>
-  </xacro:macro>
   <xacro:macro name="outer_knuckle" params="prefix fingerprefix">
     <link name="${prefix}${fingerprefix}_outer_knuckle">
@@ -146,4 +116,5 @@
     </joint>
   </xacro:macro>
+  <xacro:include filename="$(find onrobot_rg_description)/urdf/onrobot_rg6.xacro" />
   <xacro:macro name="finger_joint" params="prefix">
     <joint name="${prefix}finger_joint" type="revolute">
@@ -167,21 +138,4 @@
     <xacro:finger_joints prefix="${prefix}" fingerprefix="right" reflect="-1.0"/>
   </xacro:macro>
-  <xacro:macro name="finger_joints" params="prefix fingerprefix reflect">
-    <xacro:inner_knuckle_joint prefix="${prefix}" fingerprefix="${fingerprefix}" reflect="${reflect}"/>
-    <xacro:inner_finger_joint prefix="${prefix}" fingerprefix="${fingerprefix}"/>
-  </xacro:macro>
-  <xacro:macro name="finger_links" params="prefix fingerprefix">
-    <xacro:outer_knuckle prefix="${prefix}" fingerprefix="${fingerprefix}"/>
-    <xacro:inner_knuckle prefix="${prefix}" fingerprefix="${fingerprefix}"/>
-    <xacro:inner_finger prefix="${prefix}" fingerprefix="${fingerprefix}"/>
-  </xacro:macro>
-  <xacro:macro name="grip_target_frame" params="prefix">
-    <joint name="${prefix}grip_target_frame_joint" type="fixed">
-      <origin xyz="0 0 0.25" rpy="0 0 0" />
-      <parent link="${prefix}onrobot_rg6_base_link" />
-      <child link="${prefix}grip_target_frame" />
-    </joint>
-    <link name="${prefix}grip_target_frame"/>
-  </xacro:macro>
   <xacro:macro name="onrobot_rg6" params="prefix">
     <xacro:onrobot_rg6_base_link prefix="${prefix}"/>
@@ -192,5 +146,4 @@
     <xacro:onrobot_rg6_transmission prefix="${prefix}"/>
     <xacro:onrobot_rg6_gazebo prefix="${prefix}"/>
-    <xacro:grip_target_frame prefix="${prefix}"/>
   </xacro:macro>
 </robot>
