Commit message: Experiment ready

File: onrobot_rg_description/urdf/onrobot_rg2_model_macro.xacro (robot description, xacro)
@@ -98,5 +98,5 @@
   </xacro:macro>
   <xacro:macro name="inner_knuckle_joint" params="prefix fingerprefix reflect">
-    <joint name="${prefix}${fingerprefix}_inner_knuckle_joint" type="revolute">
+    <joint name="${prefix}${fingerprefix}_inner_knuckle_joint" type="fixed">
       <origin xyz="0 ${reflect * -0.007678} 0.1422970" rpy="0 0 ${(reflect - 1) * pi / 2}" />
       <parent link="${prefix}onrobot_rg2_base_link" />
@@ -108,5 +108,5 @@
   </xacro:macro>
   <xacro:macro name="inner_finger_joint" params="prefix fingerprefix">
-    <joint name="${prefix}${fingerprefix}_inner_finger_joint" type="revolute">
+    <joint name="${prefix}${fingerprefix}_inner_finger_joint" type="fixed">
       <origin xyz="0 ${-(0.056770-0.017178)} ${0.163974-0.125797}" rpy="0 0 0" />
       <parent link="${prefix}${fingerprefix}_outer_knuckle" />
@@ -119,5 +119,5 @@
   <xacro:include filename="$(find onrobot_rg_description)/urdf/onrobot_rg2.xacro" />
   <xacro:macro name="finger_joint" params="prefix">
-    <joint name="${prefix}finger_joint" type="revolute">
+    <joint name="${prefix}finger_joint" type="fixed">
       <origin xyz="0 -0.017178 0.125797" rpy="0 0 0" />
       <parent link="${prefix}onrobot_rg2_base_link" />
@@ -129,5 +129,5 @@
   </xacro:macro>
   <xacro:macro name="right_outer_knuckle_joint" params="prefix">
-    <joint name="${prefix}right_outer_knuckle_joint" type="revolute">
+    <joint name="${prefix}right_outer_knuckle_joint" type="fixed">
       <origin xyz="0 0.017178 0.125797" rpy="0 0 ${pi}" />
       <parent link="${prefix}onrobot_rg2_base_link" />
